Commit message: p/nodejs/client ~ UI 변경

File: production/pose_estimation_gui/server/cona.urdf (robot description, URDF)
Before this commit: robot cona, 6 links, 5 joints
Joints:
- joint robot2depth: origin xyz=0.486565500497818 0.18227818608283997 0.7440879940986633 rpy=0.6749493595139036 -0.6746417799104607 -0.20821323432433433 -> xyz=undefined undefined undefined rpy=undefined undefined undefined
- joint robot2laser1: origin xyz=1.262939453125 -0.32464599609375 0 rpy=0 0 0.00026835500871909767 -> xyz=undefined undefined undefined rpy=undefined undefined undefined
- joint robot2laser2: origin xyz=-4.294921875 -4.3502197265625 0 rpy=0 0 0.0009117726486674888 -> xyz=undefined undefined undefined rpy=undefined undefined undefined

Commit message: p/*/* ~ 부분 에러 수정

File: production/pose_estimation_gui/server/cona.urdf (robot description, URDF)
Before this commit: robot cona, 6 links, 5 joints
Joints:
- joint robot2depth: origin xyz=undefined undefined undefined rpy=undefined undefined undefined -> xyz=0.0172 -0.007 0.8882 rpy=-0.004 0.5729 -0.001
- joint robot2laser1: origin xyz=undefined undefined undefined rpy=undefined undefined undefined -> xyz=0 0 0 rpy=0 0 0
- joint robot2laser2: origin xyz=undefined undefined undefined rpy=undefined undefined undefined -> xyz=0 0 0 rpy=0 0 0
