Commit message: p/*/* ~ 핵심 기능 완성

File: production/pose_estimation_gui/server/cona_backup.urdf (robot description, URDF)
Before this commit: robot cona, 7 links, 6 joints
Links:
- removed link rgb_link
Joints:
- removed joint robot2rgb
- joint robot2depth: origin xyz=0.2645 0.0109 0.8977 rpy=-0.009 0.5762 0.0168 -> xyz=0.35 0.105 0.9 rpy=0 0.58 0
- joint robot2laser1: origin xyz=0.134 -0.001 0 rpy=0 0 -0.003 -> xyz=0.17 0 0 rpy=0 0 0
- joint robot2laser2: origin xyz=-0.147 -0.003 0 rpy=0 0 3.1336 -> xyz=-0.17 0 0 rpy=0 0 3.14
