Commit message: REST API, Mapping 주행, 수동 주행 관련 부가 기능 추가 중(1/3)

File: pose_estimation_gui/server/cona.urdf (robot description, URDF)
Before this commit: robot cona, 7 links, 6 joints
Joints:
- joint robot2depth: origin xyz=0.2645 0.0109 0.8977 rpy=-0.009 0.5762 0.0168 -> xyz=0 0 0 rpy=0 0 0
- joint robot2laser1: origin xyz=0.134 -0.001 0 rpy=0 0 -0.003 -> xyz=0 0 0 rpy=0 0 0
- joint robot2laser2: origin xyz=-0.147 -0.003 0 rpy=0 0 3.1336 -> xyz=0 0 0 rpy=0 0 0
- joint robot2rgb: origin xyz=0.2334 -0.004 1.0150 rpy=-3.135 -0.039 0.0016 -> xyz=0 0 0 rpy=0 0 0

Commit message: 통신 관련 오류 부분 수정

File: pose_estimation_gui/server/cona.urdf (robot description, URDF)
Before this commit: robot cona, 7 links, 6 joints
Joints:
- joint robot2depth: origin xyz=0 0 0 rpy=0 0 0 -> xyz=0.2639 0.0074 0.9034 rpy=-0.008 0.5796 0.0221
- joint robot2laser1: origin xyz=0 0 0 rpy=0 0 0 -> xyz=0.154 0.0002 0 rpy=0 0 -0.002
- joint robot2laser2: origin xyz=0 0 0 rpy=0 0 0 -> xyz=0 0 0 rpy=0 0 3.14
- joint robot2rgb: origin xyz=0 0 0 rpy=0 0 0 -> xyz=0.2316 -0.011 1.0085 rpy=-3.137 -0.033 -0.003
